File: KiCAD/sevenLEDboard.sch (KiCad schematic (older format))
At the start: 14 parts, among them J1 Conn_01x03_Male, U1 SC4541

Commit message: Created production 7 LED board with ZXLD1350 DC-DC bucking regulator.
Parts:
- removed C2: 10uF, Capacitor_SMD:C_0805_2012Metric, symbol Device:C
- removed R2: 2, Resistor_SMD:R_0805_2012Metric, symbol Device:R
- removed U1: SC4541, Package_TO_SOT_SMD:TSOT-23-6, symbol IRheating:SC4541
- added D8: D_Schottky, Diode_SMD:D_SOD-323, symbol Device:D_Schottky
- added U1: ZXLD1350, Package_TO_SOT_SMD:TSOT-23-5, symbol IRheating:ZXLD1350
- R1: value 10k -> 1
Other:
- moved on the sheet: C1, D1, D2, D3, D4, D5, D6, D7, J1, L1, R1
